Commit message: urdf file for iris_base is parsing, gazebo plugins not yet tested

File: ros_packages/src/uav/gazebo_model/models/iris_base/iris_base.urdf (robot description, URDF)
Before this commit: robot iris_base, 0 links, 0 joints
Links:
- added link /imu_link, mass 0.015
- added link base_link, mass 1.5; collision box size=0.47 0.47 0.11; visual mesh filename=package://uav/meshes/iris_base/iris.stl scale=1 1 1
- added link gps_link, mass 0.01; collision cylinder length=0.002 radius=0.01; visual cylinder length=0.002 radius=0.01
- added link rotor_0, mass 0.005; collision cylinder length=0.005 radius=0.128; visual mesh filename=package://uav/meshes/iris_base/iris_prop_ccw.dae scale=1 1 1
- added link rotor_1, mass 0.005; collision cylinder length=0.005 radius=0.128; visual mesh filename=package://uav/meshes/iris_base/iris_prop_ccw.dae scale=1 1 1
- added link rotor_2, mass 0.005; collision cylinder length=0.005 radius=0.128; visual mesh filename=package://uav/meshes/iris_base/iris_prop_cw.dae scale=1 1 1
- added link rotor_3, mass 0.005; collision cylinder length=0.005 radius=0.128; visual mesh filename=package://uav/meshes/iris_base/iris_prop_cw.dae scale=1 1 1
Joints:
- added joint /imu_joint: type revolute, parent base_link, child /imu_link, limit lower=0.0 upper=0.0 effort=30 velocity=0.0
- added joint gps_joint: type fixed, parent base_link, child gps_link, origin xyz=0.03 0.03 0.03 rpy=0 0 0
- added joint rotor_0_joint: type revolute, parent base_link, child rotor_0, limit effort=1e+16 velocity=1e+16
- added joint rotor_1_joint: type revolute, parent base_link, child rotor_1, limit effort=1e+16 velocity=1e+16
- added joint rotor_2_joint: type revolute, parent base_link, child rotor_2, limit effort=1e+16 velocity=1e+16
- added joint rotor_3_joint: type revolute, parent base_link, child rotor_3, limit effort=1e+16 velocity=1e+16

File: ros_packages/src/uav/gazebo_model/models/iris_base/iris_base.urdf.xacro (robot description, xacro)
@@ -1,6 +1,9 @@
-<?xml version="1.0"?>
-<robot xmlns:xacro="http://www.ros.org/wiki/xacro" name="iris_base">
+<?xml version="1.0" encoding="UTF-8"?>
+<robot name="iris_base" xmlns:xacro="http://www.ros.org/wiki/xacro">
+  <xacro:include filename="$(find uav)/gazebo_model/models/iris_base/common_properties.xacro"/>
   <!-- Main quadrotor link -->
+  <!--
   <xacro:macro name="iris_base_macro">
+  -->
     <link name="base_link">
       <inertial>
@@ -68,5 +71,5 @@
     <joint name="rotor_0_joint" type="revolute">
       <parent link="base_link"/>
-      <child link="rotor_0_joint"/>
+      <child link="rotor_0"/>
       <limit effort="1e+16" velocity="1e+16" />
     </joint>
@@ -96,5 +99,5 @@
     <joint name="rotor_1_joint" type="revolute">
       <parent link="base_link"/>
-      <child link="rotor_1_joint"/>
+      <child link="rotor_1"/>
       <limit effort="1e+16" velocity="1e+16" />
     </joint>
@@ -124,5 +127,5 @@
     <joint name="rotor_2_joint" type="revolute">
       <parent link="base_link"/>
-      <child link="rotor_2_joint"/>
+      <child link="rotor_2"/>
       <limit effort="1e+16" velocity="1e+16" />
     </joint>
@@ -152,5 +155,5 @@
     <joint name="rotor_3_joint" type="revolute">
       <parent link="base_link"/>
-      <child link="rotor_3_joint"/>
+      <child link="rotor_3"/>
       <limit effort="1e+16" velocity="1e+16" />
     </joint>
@@ -380,4 +383,4 @@
       </plugin>
     </gazebo>
-  </xacro:macro>
+  <!-- </xacro:macro> -->
 </robot>

File: ros_packages/src/uav/urdf/gps_sensor.urdf.xacro (robot description, xacro)
@@ -2,5 +2,7 @@
 <robot xmlns:xacro="http://www.ros.org/wiki/xacro">
 <xacro:macro name="gps_sensor" params="name parent *origin">
+  <!--
   <link name="gps_link"/>
+  -->
   <joint name="${name}_joint" type="fixed">
     <xacro:insert_block name="origin" />
@@ -43,3 +45,4 @@
     </sensor>
   </gazebo>
+</xacro:macro>
 </robot>
