Commit message: urdf iris_base works with iris_rplidar also for visualisation in rviz

File: ros_packages/src/uav/urdf/iris_base.urdf.xacro (robot description, xacro)
@@ -17,4 +17,5 @@
           <mesh filename="package://uav/meshes/iris_base/iris.stl" scale="1 1 1"/>
         </geometry>
+        <material name="grey"/>
       </visual>
       <collision>
@@ -58,7 +59,5 @@
           <mesh filename="package://uav/meshes/iris_base/iris_prop_ccw.dae" scale="1 1 1"/>
         </geometry>
-        <material name="blue">
-          <color rgba="0 0 .8 1"/>
-        </material>
+        <material name="blue"/>
       </visual>
       <collision>
@@ -86,7 +85,5 @@
           <mesh filename="package://uav/meshes/iris_base/iris_prop_ccw.dae" scale="1 1 1"/>
         </geometry>
-        <material name="black">
-          <color rgba="0 0 0 1"/>
-        </material>
+        <material name="black"/>
       </visual>
       <collision>
@@ -114,7 +111,5 @@
           <mesh filename="package://uav/meshes/iris_base/iris_prop_cw.dae" scale="1 1 1"/>
         </geometry>
-        <material name="blue">
-          <color rgba="0 0 .8 1"/>
-        </material>
+        <material name="blue"/>
       </visual>
       <collision>
@@ -142,7 +137,5 @@
           <mesh filename="package://uav/meshes/iris_base/iris_prop_cw.dae" scale="1 1 1"/>
         </geometry>
-        <material name="black">
-          <color rgba="0 0 0 1"/>
-        </material>
+        <material name="black"/>
       </visual>
       <collision>
